Commit message: Add param for rotation of tool changer

File: robotiq_85_description/urdf/tool_changer.urdf.xacro (robot description, xacro)
@@ -1,5 +1,5 @@
 <?xml version="1.0" encoding="utf-8"?>
 <robot xmlns:xacro="http://ros.org/wiki/xacro">
-  <xacro:macro name="tool_changer" params="prefix connected_to">
+  <xacro:macro name="tool_changer" params="prefix connected_to rotation">
     <joint name="${prefix}tool_changer_joint" type="fixed">
       <!-- The parent link must be read from the robot model it is attached to. -->
@@ -7,5 +7,5 @@
       <child link="${prefix}tool_changer_link"/>
       <!-- Adjust the origin a little to make the tool changer origin to coincide the parent link origin. -->
-      <origin xyz="0 0 -0.006" rpy="0 0 ${pi/2.0}"/>
+      <origin xyz="0 0 -0.006" rpy="0 0 ${rotation}"/>
     </joint>
     <link name="${prefix}tool_changer_link">

Commit message: Use arg forwarding to not destroy URDFs that don't include this new arg

File: robotiq_85_description/urdf/tool_changer.urdf.xacro (robot description, xacro)
@@ -1,5 +1,5 @@
 <?xml version="1.0" encoding="utf-8"?>
 <robot xmlns:xacro="http://ros.org/wiki/xacro">
-  <xacro:macro name="tool_changer" params="prefix connected_to rotation">
+  <xacro:macro name="tool_changer" params="prefix connected_to rotation:=^|0">
     <joint name="${prefix}tool_changer_joint" type="fixed">
       <!-- The parent link must be read from the robot model it is attached to. -->

Commit message: Make default rotation pi/2

File: robotiq_85_description/urdf/tool_changer.urdf.xacro (robot description, xacro)
@@ -1,5 +1,5 @@
 <?xml version="1.0" encoding="utf-8"?>
 <robot xmlns:xacro="http://ros.org/wiki/xacro">
-  <xacro:macro name="tool_changer" params="prefix connected_to rotation:=^|0">
+  <xacro:macro name="tool_changer" params="prefix connected_to rotation:=^|${pi/2.0}">
     <joint name="${prefix}tool_changer_joint" type="fixed">
       <!-- The parent link must be read from the robot model it is attached to. -->
