Commit message: Adjust description to support ros2_control.

File: robotiq_85_description/urdf/robotiq_85_gripper.transmission.xacro (robot description, xacro)
@@ -12,37 +12,4 @@
             </actuator>
         </transmission>
-        <gazebo>
-                <!-- loading plugin: mimic joints works in gazebo now -->
-            <plugin filename="libroboticsgroup_gazebo_mimic_joint_plugin.so" name="${prefix}mimic_robotiq_85_1">
-                <joint>${prefix}robotiq_85_left_knuckle_joint</joint>
-                <mimicJoint>${prefix}robotiq_85_right_knuckle_joint</mimicJoint>
-                <!--multiplier>1.0</multiplier>
-                <offset>0.0</offset-->
-            </plugin>
-            <plugin filename="libroboticsgroup_gazebo_mimic_joint_plugin.so" name="${prefix}mimic_robotiq_85_2">
-                <joint>${prefix}robotiq_85_left_knuckle_joint</joint>
-                <mimicJoint>${prefix}robotiq_85_left_inner_knuckle_joint</mimicJoint>
-                <!--multiplier>1.0</multiplier>
-                <offset>0.0</offset-->
-            </plugin>
-            <plugin filename="libroboticsgroup_gazebo_mimic_joint_plugin.so" name="${prefix}mimic_robotiq_85_3">
-                <joint>${prefix}robotiq_85_left_knuckle_joint</joint>
-                <mimicJoint>${prefix}robotiq_85_right_inner_knuckle_joint</mimicJoint>
-                <!--multiplier>1.0</multiplier>
-                <offset>0.0</offset-->
-            </plugin>
-            <plugin filename="libroboticsgroup_gazebo_mimic_joint_plugin.so" name="${prefix}mimic_robotiq_85_4">
-                <joint>${prefix}robotiq_85_left_knuckle_joint</joint>
-                <mimicJoint>${prefix}robotiq_85_left_finger_tip_joint</mimicJoint>
-                <multiplier>-1.0</multiplier>
-                <offset>0.0</offset>
-            </plugin>
-            <plugin filename="libroboticsgroup_gazebo_mimic_joint_plugin.so" name="${prefix}mimic_robotiq_85_5">
-                <joint>${prefix}robotiq_85_left_knuckle_joint</joint>
-                <mimicJoint>${prefix}robotiq_85_right_finger_tip_joint</mimicJoint>
-                <multiplier>-1.0</multiplier>
-                <offset>0.0</offset>
-            </plugin>
-        </gazebo>
     </xacro:macro>
 </robot>

File: robotiq_85_description/urdf/robotiq_85_gripper_macro.urdf.xacro (robot description, xacro)
@@ -1,332 +1,441 @@
 <?xml version="1.0"?>
 <robot name="robotiq_85_gripper" xmlns:xacro="http://ros.org/wiki/xacro">
-	<xacro:include filename="$(find robotiq_85_description)/urdf/robotiq_85_gripper.transmission.xacro" />
-	<xacro:macro name="mimic_joint_plugin_gazebo" params="name_prefix parent_joint mimic_joint has_pid:=false multiplier:=1.0 offset:=0 sensitiveness:=0.0 max_effort:=1.0 robot_namespace:=''">
-		<gazebo>
-			<plugin name="${name_prefix}mimic_joint_plugin" filename="libroboticsgroup_gazebo_mimic_joint_plugin.so">
-				<joint>${parent_joint}</joint>
-				<mimicJoint>${mimic_joint}</mimicJoint>
-				<xacro:if value="${has_pid}">                     <!-- if set to true, PID parameters from "/gazebo_ros_control/pid_gains/${mimic_joint}" are loaded -->
-					<hasPID />
-				</xacro:if>
-				<multiplier>${multiplier}</multiplier>
-				<offset>${offset}</offset>
-				<sensitiveness>${sensitiveness}</sensitiveness>   <!-- if absolute difference between setpoint and process value is below this threshold, do nothing; 0.0 = disable [rad] -->
-				<maxEffort>${max_effort}</maxEffort>              <!-- only taken into account if has_pid:=true [Nm] -->
-				<xacro:unless value="${robot_namespace == ''}">
-					<robotNamespace>($robot_namespace)</robotNamespace>
-				</xacro:unless>
-			</plugin>
-		</gazebo>
-	</xacro:macro>
-	<xacro:macro name="robotiq_85_gripper" params="prefix parent *origin sim:=false">
-		<!-- The current hardware driver does not depend on ros2_control but we do utilize
-				 it for simulating the gripper in Gazebo. Enabling this on hardware causes the
-				 JointStateBroadcaster to publish values for all joints including ones that are
-				 mimic'd which is causing issues on systems consuming the joint_state data. -->
-		<xacro:if value="${sim}">
-			<!-- ros2 control include -->
-			<xacro:include filename="$(find robotiq_85_description)/urdf/robotiq_85_gripper.ros2_control.xacro"/>
-			<!-- ros2 control instance -->
-			<xacro:robotiq_85_gripper_ros2_control name="RobotiqGripperSystem"/>
-		</xacro:if>
-		<joint name="${prefix}robotiq_85_base_joint" type="fixed">
-			<parent link="${parent}"/>
-			<child link="${prefix}robotiq_85_base_link"/>
-			<xacro:insert_block name="origin"/>
-		</joint>
-		<link name="${prefix}robotiq_85_base_link">
-			<!-- Visual aid for grasping -->
-			<visual>
-				<origin xyz="0.16 0 0" rpy="0 0 0" />
-				<geometry>
-					<sphere radius="0.007"/>
-				</geometry>
-				<material name="">
-					<color rgba="0 1.0 0 1.0"/>
-				</material>
-			</visual>
-			<!-- Gripper body -->
-			<visual>
-				<geometry>
-					<mesh filename="package://robotiq_85_description/meshes/visual/robotiq_85_base_link.dae"/>
-				</geometry>
-			</visual>
-			<collision>
-				<geometry>
-					<mesh filename="package://robotiq_85_description/meshes/collision/robotiq_85_base_link.stl"/>
-				</geometry>
-			</collision>
-			<inertial>
-				<mass value="0.636951" />
-				<origin xyz="0.0 0.0 0.0" />
-				<inertia ixx = "0.000380" ixy = "0.000000" ixz = "0.000000"
-					iyx = "0.000000" iyy = "0.001110" iyz = "0.000000"
-					izx = "0.000000" izy = "0.000000" izz = "0.001171" />
-			</inertial>
-		</link>
-		<joint name="${prefix}robotiq_85_left_knuckle_joint" type="revolute">
-			<parent link="${prefix}robotiq_85_base_link"/>
-			<child link="${prefix}robotiq_85_left_knuckle_link"/>
-			<axis xyz="0 0 1"/>
-			<origin rpy="${pi} 0.0 0.0" xyz="0.05490451627 0.03060114443 0.0"/>
-			<limit lower="0.0" upper="0.804" velocity="0.5" effort="50"/>
-			<dynamics damping="100.0" />
-		</joint>
-		<gazebo reference="${prefix}robotiq_85_left_knuckle_link">
-			<kp>1000000.0</kp>
-			<kd>100.0</kd>
-			<mu1>30.0</mu1>
-			<mu2>30.0</mu2>
-			<maxVel>1.0</maxVel>
-			<minDepth>0.001</minDepth>
-			<material>Gazebo/Grey</material>
-		</gazebo>
-		<joint name="${prefix}robotiq_85_right_knuckle_joint" type="continuous">
-			<parent link="${prefix}robotiq_85_base_link"/>
-			<child link="${prefix}robotiq_85_right_knuckle_link"/>
-			<axis xyz="0 0 1"/>
-			<origin rpy="0.0 0.0 0.0" xyz="0.05490451627 -0.03060114443 0.0"/>
-			<limit lower="-3.14" upper="3.14" velocity="100.0" effort="50"/>
-			<mimic joint="${prefix}robotiq_85_left_knuckle_joint"/>
-			<dynamics damping="100.0" />
-		</joint>
-		<gazebo reference="${prefix}robotiq_85_right_knuckle_link">
-			<kp>1000000.0</kp>
-			<kd>100.0</kd>
-			<mu1>30.0</mu1>
-			<mu2>30.0</mu2>
-			<maxVel>1.0</maxVel>
-			<minDepth>0.001</minDepth>
-			<material>Gazebo/Grey</material>
-		</gazebo>
-		<xacro:mimic_joint_plugin_gazebo name_prefix="{prefix}robotiq_85_right_knuckle_joint"
-			parent_joint="${prefix}robotiq_85_left_knuckle_joint" mimic_joint="${prefix}robotiq_85_right_knuckle_joint"
-			multiplier="1.0" max_effort="10.0" />
-		<link name="${prefix}robotiq_85_left_knuckle_link">
-			<visual>
-				<geometry>
-					<mesh filename="package://robotiq_85_description/meshes/visual/robotiq_85_knuckle_link.dae"/>
-				</geometry>
-			</visual>
-			<collision>
-				<geometry>
-					<mesh filename="package://robotiq_85_description/meshes/collision/robotiq_85_knuckle_link.stl"/>
-				</geometry>
-			</collision>
-			<inertial>
-				<mass value="0.018491" />
-				<origin xyz="0.0 0.0 0.0" />
-				<inertia ixx = "0.000009" ixy = "-0.000001" ixz = "0.000000"
-					iyx = "-0.000001" iyy = "0.000001" iyz = "0.000000"
-					izx = "0.000000" izy = "0.000000" izz = "0.000010" />
-			</inertial>
-		</link>
-		<link name="${prefix}robotiq_85_right_knuckle_link">
-			<visual>
-				<geometry>
-					<mesh filename="package://robotiq_85_description/meshes/visual/robotiq_85_knuckle_link.dae"/>
-				</geometry>
-			</visual>
-			<collision>
-				<geometry>
-					<mesh filename="package://robotiq_85_description/meshes/collision/robotiq_85_knuckle_link.stl"/>
-				</geometry>
-			</collision>
-			<inertial>
-				<mass value="0.018491" />
-				<origin xyz="0.0 0.0 0.0" />
-				<inertia ixx = "0.000009" ixy = "-0.000001" ixz = "0.000000"
-					iyx = "-0.000001" iyy = "0.000001" iyz = "0.000000"
-					izx = "0.000000" izy = "0.000000" izz = "0.000010" />
-			</inertial>
-		</link>
-		<joint name="${prefix}robotiq_85_left_finger_joint" type="fixed">
-			<parent link="${prefix}robotiq_85_left_knuckle_link"/>
-			<child link="${prefix}robotiq_85_left_finger_link"/>
-			<origin xyz="-0.00408552455 -0.03148604435 0.0" rpy="0 0 0" />
-		</joint>
-		<joint name="${prefix}robotiq_85_right_finger_joint" type="fixed">
-			<parent link="${prefix}robotiq_85_right_knuckle_link"/>
-			<child link="${prefix}robotiq_85_right_finger_link"/>
-			<origin xyz="-0.00408552455 -0.03148604435 0.0" rpy="0 0 0" />
-		</joint>
-		<link name="${prefix}robotiq_85_left_finger_link">
-			<visual>
-				<geometry>
-					<mesh filename="package://robotiq_85_description/meshes/visual/robotiq_85_finger_link.dae"/>
-				</geometry>
-			</visual>
-			<collision>
-				<geometry>
-					<mesh filename="package://robotiq_85_description/meshes/collision/robotiq_85_finger_link.stl"/>
-				</geometry>
-			</collision>
-			<inertial>
-				<mass value="0.027309" />
-				<origin xyz="0.0 0.0 0.0" />
-				<inertia ixx = "0.000003" ixy = "-0.000002" ixz = "0.000000"
-					iyx = "-0.000002" iyy = "0.000021" iyz = "0.000000"
-					izx = "0.000000" izy = "0.000000" izz = "0.000020" />
-			</inertial>
-		</link>
-		<link name="${prefix}robotiq_85_right_finger_link">
-			<visual>
-				<geometry>
-					<mesh filename="package://robotiq_85_description/meshes/visual/robotiq_85_finger_link.dae"/>
-				</geometry>
-			</visual>
-			<collision>
-				<geometry>
-					<mesh filename="package://robotiq_85_description/meshes/collision/robotiq_85_finger_link.stl"/>
-				</geometry>
-			</collision>
-			<inertial>
-				<mass value="0.027309" />
-				<origin xyz="0.0 0.0 0.0" />
-				<inertia ixx = "0.000003" ixy = "-0.000002" ixz = "0.000000"
-					iyx = "-0.000002" iyy = "0.000021" iyz = "0.000000"
-					izx = "0.000000" izy = "0.000000" izz = "0.000020" />
-			</inertial>
-		</link>
-		<joint name="${prefix}robotiq_85_left_inner_knuckle_joint" type="continuous">
-			<parent link="${prefix}robotiq_85_base_link"/>
-			<child link="${prefix}robotiq_85_left_inner_knuckle_link"/>
-			<axis xyz="0 0 1"/>
-			<origin xyz="0.06142 0.0127 0" rpy="${pi} 0.0 0.0" />
-			<limit lower="-3.14" upper="3.14" velocity="100.0" effort="0.1"/>
-			<mimic joint="${prefix}robotiq_85_left_knuckle_joint" offset="0"/>
-		</joint>
-		<xacro:mimic_joint_plugin_gazebo name_prefix="${prefix}robotiq_85_left_inner_knuckle_joint"
-			parent_joint="${prefix}robotiq_85_left_knuckle_joint" mimic_joint="${prefix}robotiq_85_left_inner_knuckle_joint"
-			multiplier="1.0" max_effort="10.0" />
-		<joint name="${prefix}robotiq_85_right_inner_knuckle_joint" type="continuous">
-			<parent link="${prefix}robotiq_85_base_link"/>
-			<child link="${prefix}robotiq_85_right_inner_knuckle_link"/>
-			<axis xyz="0 0 1"/>
-			<origin xyz="0.06142 -0.0127 0" rpy="0 0 0"/>
-			<limit lower="-3.14" upper="3.14" velocity="100.0" effort="0.1"/>
-			<mimic joint="${prefix}robotiq_85_left_knuckle_joint" offset="0"/>
-		</joint>
-		<xacro:mimic_joint_plugin_gazebo name_prefix="${prefix}robotiq_85_right_inner_knuckle_joint"
-			parent_joint="${prefix}robotiq_85_left_knuckle_joint" mimic_joint="${prefix}robotiq_85_right_inner_knuckle_joint"
-			multiplier="1.0" max_effort="10.0" />
-		<link name="${prefix}robotiq_85_left_inner_knuckle_link">
-			<visual>
-				<geometry>
-					<mesh filename="package://robotiq_85_description/meshes/visual/robotiq_85_inner_knuckle_link.dae"/>
-				</geometry>
-			</visual>
-			<collision>
-				<geometry>
-					<mesh filename="package://robotiq_85_description/meshes/collision/robotiq_85_inner_knuckle_link.stl"/>
-				</geometry>
-			</collision>
-			<inertial>
-				<mass value="0.029951" />
-				<origin xyz="0.0 0.0 0.0" />
-				<inertia ixx = "0.000039" ixy = "0.000000" ixz = "0.000000"
-					iyx = "0.000000" iyy = "0.000005" iyz = "0.000000"
-					izx = "0.000000" izy = "0.000000" izz = "0.000035" />
-			</inertial>
-		</link>
-		<link name="${prefix}robotiq_85_right_inner_knuckle_link">
-			<visual>
-				<geometry>
-					<mesh filename="package://robotiq_85_description/meshes/visual/robotiq_85_inner_knuckle_link.dae"/>
-				</geometry>
-			</visual>
-			<collision>
-				<geometry>
-					<mesh filename="package://robotiq_85_description/meshes/collision/robotiq_85_inner_knuckle_link.stl"/>
-				</geometry>
-			</collision>
-			<inertial>
-				<mass value="0.029951" />
-				<origin xyz="0.0 0.0 0.0" />
-				<inertia ixx = "0.000039" ixy = "0.000000" ixz = "0.000000"
-					iyx = "0.000000" iyy = "0.000005" iyz = "0.000000"
-					izx = "0.000000" izy = "0.000000" izz = "0.000035" />
-			</inertial>
-		</link>
-		<joint name="${prefix}robotiq_85_left_finger_tip_joint" type="continuous">
-			<parent link="${prefix}robotiq_85_left_inner_knuckle_link"/>
-			<child link="${prefix}robotiq_85_left_finger_tip_link"/>
-			<axis xyz="0 0 1"/>
-			<origin xyz="0.04303959807 -0.03759940821 0.0" rpy="0.0 0.0 0.0"/>
-			<limit lower="-3.14" upper="3.14" velocity="100.0" effort="0.1"/>
-			<mimic joint="${prefix}robotiq_85_left_knuckle_joint" multiplier="-1"/>
-		</joint>
-		<xacro:mimic_joint_plugin_gazebo name_prefix="${prefix}robotiq_85_left_finger_tip_joint"
-			parent_joint="${prefix}robotiq_85_left_knuckle_joint" mimic_joint="${prefix}robotiq_85_left_finger_tip_joint"
-			multiplier="1.0" max_effort="10.0" />
-		<joint name="${prefix}robotiq_85_right_finger_tip_joint" type="continuous">
-			<parent link="${prefix}robotiq_85_right_inner_knuckle_link"/>
-			<child link="${prefix}robotiq_85_right_finger_tip_link"/>
-			<axis xyz="0 0 1"/>
-			<origin rpy="0.0 0.0 0.0" xyz="0.04303959807 -0.03759940821  0.0"/>
-			<limit lower="-3.14" upper="3.14" velocity="100.0" effort="0.1"/>
-			<mimic joint="${prefix}robotiq_85_left_knuckle_joint" multiplier="-1"/>
-		</joint>
-		<xacro:mimic_joint_plugin_gazebo name_prefix="${prefix}robotiq_85_right_finger_tip_joint"
-			parent_joint="${prefix}robotiq_85_left_knuckle_joint" mimic_joint="${prefix}robotiq_85_right_finger_tip_joint"
-			multiplier="1.0" max_effort="10.0" />
-		<link name="${prefix}robotiq_85_left_finger_tip_link">
-			<visual>
-				<geometry>
-					<mesh filename="package://robotiq_85_description/meshes/visual/robotiq_85_finger_tip_link.dae"/>
-				</geometry>
-			</visual>
-			<collision>
-				<geometry>
-					<mesh filename="package://robotiq_85_description/meshes/collision/robotiq_85_finger_tip_link.stl"/>
-				</geometry>
-			</collision>
-			<inertial>
-				<mass value="0.019555" />
-				<origin xyz="0.0 0.0 0.0" />
-				<inertia ixx = "0.000002" ixy = "0.000000" ixz = "0.000000"
-					iyx = "0.000000" iyy = "0.000005" iyz = "0.000000"
-					izx = "0.000000" izy = "0.000000" izz = "0.000006" />
-			</inertial>
-		</link>
-		<gazebo reference="${prefix}robotiq_85_left_finger_tip_link">
-			<kp>1000000.0</kp>
-			<kd>100.0</kd>
-			<mu1>30.0</mu1>
-			<mu2>30.0</mu2>
-			<maxVel>1.0</maxVel>
-			<minDepth>0.001</minDepth>
-			<material>Gazebo/Grey</material>
-		</gazebo>
-		<link name="${prefix}robotiq_85_right_finger_tip_link">
-			<visual>
-				<geometry>
-					<mesh filename="package://robotiq_85_description/meshes/visual/robotiq_85_finger_tip_link.dae"/>
-				</geometry>
-			</visual>
-			<collision>
-				<geometry>
-					<mesh filename="package://robotiq_85_description/meshes/collision/robotiq_85_finger_tip_link.stl"/>
-				</geometry>
-			</collision>
-			<inertial>
-				<mass value="0.019555" />
-				<origin xyz="0.0 0.0 0.0" />
-				<inertia ixx = "0.000002" ixy = "0.000000" ixz = "0.000000"
-					iyx = "0.000000" iyy = "0.000005" iyz = "0.000000"
-					izx = "0.000000" izy = "0.000000" izz = "0.000006" />
-			</inertial>
-		</link>
-		<gazebo reference="${prefix}robotiq_85_right_finger_tip_link">
-			<kp>1000000.0</kp>
-			<kd>100.0</kd>
-			<mu1>30.0</mu1>
-			<mu2>30.0</mu2>
-			<maxVel>1.0</maxVel>
-			<minDepth>0.001</minDepth>
-			<material>Gazebo/Grey</material>
-		</gazebo>
-		<xacro:robotiq_85_gripper_transmission prefix="${prefix}" />
-	</xacro:macro>
+  <xacro:include filename="$(find robotiq_85_description)/urdf/robotiq_85_gripper.transmission.xacro" />
+  <xacro:macro name="robotiq_85_gripper" params="
+    name
+    prefix
+    parent
+    *origin
+    use_fake_hardware:=false
+    fake_sensor_commands:=false
+    gazebo_sim:=false
+    ignition_sim:=false
+    use_ros2_control:=false">
+    <!-- The current hardware driver does not depend on ros2_control but we do utilize
+    it for simulating the gripper in Gazebo. Enabling this on hardware causes the
+    JointStateBroadcaster to publish values for all joints including ones that are
+    mimic'd which is causing issues on systems consuming the joint_state data. -->
+    <xacro:if value="${use_ros2_control}">
+      <!-- ros2 control include -->
+      <xacro:include filename="$(find robotiq_85_description)/urdf/robotiq_85_gripper.ros2_control.xacro"/>
+      <!-- ros2 control instance -->
+      <xacro:robotiq_85_gripper_ros2_control name="RobotiqGripperSystem"/>
+    </xacro:if>
+    <joint name="${prefix}robotiq_85_base_joint" type="fixed">
+      <parent link="${parent}"/>
+      <child link="${prefix}robotiq_85_base_link"/>
+      <xacro:insert_block name="origin"/>
+    </joint>
+    <link name="${prefix}robotiq_85_base_link">
+      <!-- Visual aid for grasping -->
+      <visual>
+        <origin xyz="0.16 0 0" rpy="0 0 0" />
+        <geometry>
+          <sphere radius="0.007"/>
+        </geometry>
+        <material name="">
+          <color rgba="0 1.0 0 1.0"/>
+        </material>
+      </visual>
+      <!-- Gripper body -->
+      <visual>
+        <geometry>
+          <mesh filename="file://$(find robotiq_85_description)/meshes/visual/robotiq_85_base_link.dae"/>
+        </geometry>
+      </visual>
+      <collision>
+        <geometry>
+          <mesh filename="file://$(find robotiq_85_description)/meshes/collision/robotiq_85_base_link.stl"/>
+        </geometry>
+      </collision>
+      <inertial>
+        <mass value="0.636951" />
+        <origin xyz="0.0 0.0 0.0" />
+        <inertia ixx = "0.000380" ixy = "0.000000" ixz = "0.000000"
+          iyx = "0.000000" iyy = "0.001110" iyz = "0.000000"
+          izx = "0.000000" izy = "0.000000" izz = "0.001171" />
+      </inertial>
+    </link>
+    <joint name="${prefix}robotiq_85_left_knuckle_joint" type="revolute">
+      <parent link="${prefix}robotiq_85_base_link"/>
+      <child link="${prefix}robotiq_85_left_knuckle_link"/>
+      <axis xyz="0 0 1"/>
+      <origin rpy="${pi} 0.0 0.0" xyz="0.05490451627 0.03060114443 0.0"/>
+      <limit lower="0.0" upper="0.804" velocity="0.5" effort="50"/>
+      <dynamics damping="100.0" />
+    </joint>
+    <gazebo reference="${prefix}robotiq_85_left_knuckle_link">
+      <kp>1000000.0</kp>
+      <kd>100.0</kd>
+      <mu1>30.0</mu1>
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