Commit message: Make ros_control optional

File: robotiq_85_description/urdf/robotiq_85_gripper_macro.urdf.xacro (robot description, xacro)
@@ -20,9 +20,11 @@
 		</gazebo>
 	</xacro:macro>
-	<xacro:macro name="robotiq_85_gripper" params="prefix parent *origin">
-		<!-- ros2 control include -->
-		<xacro:include filename="$(find robotiq_85_description)/urdf/robotiq_85_gripper.ros2_control.xacro"/>
-		<!-- ros2 control instance -->
-		<xacro:robotiq_85_gripper_ros2_control name="RobotiqGripperSystem"/>
+	<xacro:macro name="robotiq_85_gripper" params="prefix parent *origin sim:=false">
+		<xacro:if value="${sim}">
+			<!-- ros2 control include -->
+			<xacro:include filename="$(find robotiq_85_description)/urdf/robotiq_85_gripper.ros2_control.xacro"/>
+			<!-- ros2 control instance -->
+			<xacro:robotiq_85_gripper_ros2_control name="RobotiqGripperSystem"/>
+		</xacro:if>
 		<joint name="${prefix}robotiq_85_base_joint" type="fixed">
 			<parent link="${parent}"/>

Commit message: Remove visual aid in sim. Change mesh paths for gripper adapter.

File: robotiq_85_description/urdf/robotiq_85_gripper_macro.urdf.xacro (robot description, xacro)
@@ -33,14 +33,16 @@
     </joint>
     <link name="${prefix}robotiq_85_base_link">
-      <!-- Visual aid for grasping -->
-      <visual>
-        <origin xyz="0.16 0 0" rpy="0 0 0" />
-        <geometry>
-          <sphere radius="0.007"/>
-        </geometry>
-        <material name="">
-          <color rgba="0 1.0 0 1.0"/>
-        </material>
-      </visual>
+      <xacro:unless value="${sim_ignition}">
+        <!-- Visual aid for grasping -->
+        <visual>
+          <origin xyz="0.16 0 0" rpy="0 0 0" />
+          <geometry>
+            <sphere radius="0.007"/>
+          </geometry>
+          <material name="">
+            <color rgba="0 1.0 0 1.0"/>
+          </material>
+        </visual>
+      </xacro:unless>
       <!-- Gripper body -->
       <visual>

File: robotiq_85_description/urdf/ur_to_robotiq_adapter.urdf.xacro (robot description, xacro)
@@ -12,5 +12,5 @@
           <origin xyz="0 0 0" rpy="0 0 0" />
           <geometry>
-            <mesh filename="package://robotiq_85_description/meshes/visual/ur_to_robotiq_adapter.dae"/>
+            <mesh filename="file://$(find robotiq_85_description)/meshes/visual/ur_to_robotiq_adapter.dae"/>
           </geometry>
         </visual>
@@ -18,5 +18,5 @@
           <origin xyz="0 0 0" rpy="0 0 0"/>
           <geometry>
-            <mesh filename="package://robotiq_85_description/meshes/collision/ur_to_robotiq_adapter.stl"/>
+            <mesh filename="file://$(find robotiq_85_description)/meshes/collision/ur_to_robotiq_adapter.stl"/>
           </geometry>
         </collision>
