Commit message: ros2_control part is moved to .ros2_control.xacro file.

File: robotiq_85_description/urdf/robotiq_85_gripper.ros2_control.xacro (robot description, xacro)
@@ -1,51 +1,144 @@
 <?xml version="1.0"?>
 <robot xmlns:xacro="http://www.ros.org/wiki/xacro">
-    <xacro:macro name="robotiq_85_gripper_ros2_control" params="name">
-        <ros2_control name="${name}" type="system">
-            <hardware>
-                <plugin>fake_components/GenericSystem</plugin>
-            </hardware>
-            <joint name="robotiq_85_left_knuckle_joint">
-                <param name="initial_position">0.7929</param>
-                <command_interface name="position" />
-                <state_interface name="position"/>
-                <state_interface name="velocity"/>
-            </joint>
-            <joint name="robotiq_85_right_knuckle_joint">
-                <param name="mimic">robotiq_85_left_knuckle_joint</param>
-                <param name="multiplier">1</param>
-                <command_interface name="position" />
-                <state_interface name="position"/>
-                <state_interface name="velocity"/>
-            </joint>
-            <joint name="robotiq_85_left_inner_knuckle_joint">
-                <param name="mimic">robotiq_85_left_knuckle_joint</param>
-                <param name="multiplier">1</param>
-                <command_interface name="position" />
-                <state_interface name="position"/>
-                <state_interface name="velocity"/>
-            </joint>
-            <joint name="robotiq_85_right_inner_knuckle_joint">
-                <param name="mimic">robotiq_85_left_knuckle_joint</param>
-                <param name="multiplier">1</param>
-                <command_interface name="position" />
-                <state_interface name="position"/>
-                <state_interface name="velocity"/>
-            </joint>
-            <joint name="robotiq_85_left_finger_tip_joint">
-                <param name="mimic">robotiq_85_left_knuckle_joint</param>
-                <param name="multiplier">-1</param>
-                <command_interface name="position" />
-                <state_interface name="position"/>
-                <state_interface name="velocity"/>
-            </joint>
-            <joint name="robotiq_85_right_finger_tip_joint">
-                <param name="mimic">robotiq_85_left_knuckle_joint</param>
-                <param name="multiplier">-1</param>
-                <command_interface name="position" />
-                <state_interface name="position"/>
-                <state_interface name="velocity"/>
-            </joint>
-        </ros2_control>
-    </xacro:macro>
+  <xacro:macro name="robotiq_85_gripper_ros2_control" params="
+    name
+    prefix
+    use_fake_hardware:=false
+    fake_sensor_commands:=false
+    sim_gazebo:=false
+    sim_ignition:=false">
+<!-- NOTE - currently using "system" because it is only supported hardware_interface-type by Gazebo and Ignition -->
+    <ros2_control name="${name}" type="system">
+      <hardware>
+        <xacro:if value="${sim_gazebo}">
+          <plugin>gazebo_ros2_control/GazeboSystem</plugin>
+        </xacro:if>
+        <xacro:if value="${sim_ignition}">
+          <plugin>ignition_ros2_control/IgnitionSystem</plugin>
+        </xacro:if>
+        <xacro:if value="${use_fake_hardware}">
+          <plugin>fake_components/GenericSystem</plugin>
+          <param name="fake_sensor_commands">${fake_sensor_commands}</param>
+          <param name="state_following_offset">0.0</param>
+        </xacro:if>
+        <xacro:unless value="${use_fake_hardware or sim_gazebo or sim_ignition}">
+          <plugin>robotiq_hardware_interface/NOT_IMPLEMENTED_YET</plugin>
+          <param name="ADD_GRIPPER_RELEVANT_PARAMETERS">654321</param>
+        </xacro:unless>
+      </hardware>
+      <joint name="${prefix}robotiq_85_left_knuckle_joint">
+        <param name="initial_position">0.7929</param>
+        <command_interface name="position">
+          <param name="min">0.0</param>
+          <param name="max">0.085</param>
+        </command_interface>
+        <command_interface name="velocity">
+          <param name="min">0.013</param>
+          <param name="max">0.1</param>
+        </command_interface>
+        <command_interface name="force">
+          <param name="min">5.0</param>
+          <param name="max">220.0</param>
+        </command_interface>
+        <state_interface name="position"/>
+        <state_interface name="velocity"/>
+        <state_interface name="force"/>
+      </joint>
+      <joint name="${prefix}robotiq_85_right_knuckle_joint">
+        <param name="mimic">${prefix}robotiq_85_left_knuckle_joint</param>
+        <param name="multiplier">1</param>
+        <command_interface name="position">
+          <param name="min">0.0</param>
+          <param name="max">0.085</param>
+        </command_interface>
+        <command_interface name="velocity">
+          <param name="min">0.013</param>
+          <param name="max">0.1</param>
+        </command_interface>
+        <command_interface name="force">
+          <param name="min">5.0</param>
+          <param name="max">220.0</param>
+        </command_interface>
+        <state_interface name="position"/>
+        <state_interface name="velocity"/>
+        <state_interface name="force"/>
+      </joint>
+      <joint name="${prefix}robotiq_85_left_inner_knuckle_joint">
+        <param name="mimic">${prefix}robotiq_85_left_knuckle_joint</param>
+        <param name="multiplier">1</param>
+        <command_interface name="position">
+          <param name="min">0.0</param>
+          <param name="max">0.085</param>
+        </command_interface>
+        <command_interface name="velocity">
+          <param name="min">0.013</param>
+          <param name="max">0.1</param>
+        </command_interface>
+        <command_interface name="force">
+          <param name="min">5.0</param>
+          <param name="max">220.0</param>
+        </command_interface>
+        <state_interface name="position"/>
+        <state_interface name="velocity"/>
+        <state_interface name="force"/>
+      </joint>
+      <joint name="${prefix}robotiq_85_right_inner_knuckle_joint">
+        <param name="mimic">${prefix}robotiq_85_left_knuckle_joint</param>
+        <param name="multiplier">1</param>
+        <command_interface name="position">
+          <param name="min">0.0</param>
+          <param name="max">0.085</param>
+        </command_interface>
+        <command_interface name="velocity">
+          <param name="min">0.013</param>
+          <param name="max">0.1</param>
+        </command_interface>
+        <command_interface name="force">
+          <param name="min">5.0</param>
+          <param name="max">220.0</param>
+        </command_interface>
+        <state_interface name="position"/>
+        <state_interface name="velocity"/>
+        <state_interface name="force"/>
+      </joint>
+      <joint name="${prefix}robotiq_85_left_finger_tip_joint">
+        <param name="mimic">${prefix}robotiq_85_left_knuckle_joint</param>
+        <param name="multiplier">-1</param>
+        <command_interface name="position">
+          <param name="min">0.0</param>
+          <param name="max">0.085</param>
+        </command_interface>
+        <command_interface name="velocity">
+          <param name="min">0.013</param>
+          <param name="max">0.1</param>
+        </command_interface>
+        <command_interface name="force">
+          <param name="min">5.0</param>
+          <param name="max">220.0</param>
+        </command_interface>
+        <state_interface name="position"/>
+        <state_interface name="velocity"/>
+        <state_interface name="force"/>
+      </joint>
+      <joint name="${prefix}robotiq_85_right_finger_tip_joint">
+        <param name="mimic">${prefix}robotiq_85_left_knuckle_joint</param>
+        <param name="multiplier">-1</param>
+        <command_interface name="position">
+          <param name="min">0.0</param>
+          <param name="max">0.085</param>
+        </command_interface>
+        <command_interface name="velocity">
+          <param name="min">0.013</param>
+          <param name="max">0.1</param>
+        </command_interface>
+        <command_interface name="force">
+          <param name="min">5.0</param>
+          <param name="max">220.0</param>
+        </command_interface>
+        <state_interface name="position"/>
+        <state_interface name="velocity"/>
+        <state_interface name="force"/>
+      </joint>
+    </ros2_control>
+  </xacro:macro>
 </robot>

File: robotiq_85_description/urdf/robotiq_85_gripper_macro.urdf.xacro (robot description, xacro)
@@ -2,4 +2,5 @@
 <robot name="robotiq_85_gripper" xmlns:xacro="http://ros.org/wiki/xacro">
   <xacro:include filename="$(find robotiq_85_description)/urdf/robotiq_85_gripper.transmission.xacro" />
+  <xacro:include filename="$(find robotiq_85_description)/urdf/robotiq_85_gripper.ros2_control.xacro"/>
   <xacro:macro name="robotiq_85_gripper" params="
     name
@@ -7,5 +8,4 @@
     parent
     *origin
-    use_ros2_control:=false
     use_fake_hardware:=false
     fake_sensor_commands:=false
@@ -13,12 +13,17 @@
     sim_ignition:=false">
     <!-- The current hardware driver does not depend on ros2_control but we do utilize
-    it for simulating the gripper in Gazebo. Enabling this on hardware causes the
-    JointStateBroadcaster to publish values for all joints including ones that are
-    mimic'd which is causing issues on systems consuming the joint_state data. -->
-    <xacro:if value="${use_ros2_control}">
-      <!-- ros2 control include -->
-      <xacro:include filename="$(find robotiq_85_description)/urdf/robotiq_85_gripper.ros2_control.xacro"/>
+    it for simulating the gripper with FakeSystem, Gazebo and  Igntion. Enabling this on
+    hardware causes the JointStateBroadcaster to publish values for all joints including
+    ones that are mimic'd which is causing issues on systems consuming the joint_state data. -->
+    <xacro:if value="${use_fake_hardware or sim_gazebo or sim_ignition}">
       <!-- ros2 control instance -->
-      <xacro:robotiq_85_gripper_ros2_control name="RobotiqGripperSystem"/>
+      <xacro:robotiq_85_gripper_ros2_control
+        name="${name}"
+        prefix="${prefix}"
+        use_fake_hardware="${use_fake_hardware}"
+        fake_sensor_commands="${fake_sensor_commands}"
+        sim_gazebo="${sim_gazebo}"
+        sim_ignition="${sim_ignition}"
+        />
     </xacro:if>
     <joint name="${prefix}robotiq_85_base_joint" type="fixed">
@@ -305,137 +310,4 @@
     </gazebo>-->
     <xacro:robotiq_85_gripper_transmission prefix="${prefix}" />
-    <!-- ros2_control part -->
-    <!-- NOTE - currently using "system" because it is only supported hardware_interface-type by Gazebo and Ignition -->
-    <ros2_control name="${name}" type="system">
-      <hardware>
-        <xacro:if value="${sim_gazebo}">
-          <plugin>gazebo_ros2_control/GazeboSystem</plugin>
-        </xacro:if>
-        <xacro:if value="${sim_ignition}">
-          <plugin>ignition_ros2_control/IgnitionSystem</plugin>
-        </xacro:if>
-        <xacro:if value="${use_fake_hardware}">
-          <plugin>fake_components/GenericSystem</plugin>
-          <param name="fake_sensor_commands">${fake_sensor_commands}</param>
-          <param name="state_following_offset">0.0</param>
-        </xacro:if>
-        <xacro:unless value="${use_fake_hardware or sim_gazebo or sim_ignition}">
-          <plugin>robotiq_hardware_interface/NOT_IMPLEMENTED_YET</plugin>
-          <param name="ADD_GRIPPER_RELEVANT_PARAMETERS">654321</param>
-        </xacro:unless>
-      </hardware>
-      <joint name="${prefix}robotiq_85_left_knuckle_joint">
-        <command_interface name="position">
-          <param name="min">0.0</param>
-          <param name="max">0.085</param>
-        </command_interface>
-        <command_interface name="velocity">
-          <param name="min">0.013</param>
-          <param name="max">0.1</param>
-        </command_interface>
-        <command_interface name="force">
-          <param name="min">5.0</param>
-          <param name="max">220.0</param>
-        </command_interface>
-        <state_interface name="position"/>
-        <state_interface name="velocity"/>
-        <state_interface name="force"/>
-      </joint>
-      <joint name="${prefix}robotiq_85_right_knuckle_joint">
-        <param name="mimic">${prefix}robotiq_85_left_knuckle_joint</param>
-        <param name="multiplier">1</param>
-        <command_interface name="position">
-          <param name="min">0.0</param>
-          <param name="max">0.085</param>
-        </command_interface>
-        <command_interface name="velocity">
-          <param name="min">0.013</param>
-          <param name="max">0.1</param>
-        </command_interface>
-        <command_interface name="force">
-          <param name="min">5.0</param>
-          <param name="max">220.0</param>
-        </command_interface>
-        <state_interface name="position"/>
-        <state_interface name="velocity"/>
-        <state_interface name="force"/>
-      </joint>
-      <joint name="${prefix}robotiq_85_left_inner_knuckle_joint">
-        <param name="mimic">${prefix}robotiq_85_left_knuckle_joint</param>
-        <param name="multiplier">1</param>
-        <command_interface name="position">
-          <param name="min">0.0</param>
-          <param name="max">0.085</param>
-        </command_interface>
-        <command_interface name="velocity">
-          <param name="min">0.013</param>
-          <param name="max">0.1</param>
-        </command_interface>
-        <command_interface name="force">
-          <param name="min">5.0</param>
-          <param name="max">220.0</param>
-        </command_interface>
-        <state_interface name="position"/>
-        <state_interface name="velocity"/>
-        <state_interface name="force"/>
-      </joint>
-      <joint name="${prefix}robotiq_85_right_inner_knuckle_joint">
-        <param name="mimic">${prefix}robotiq_85_left_knuckle_joint</param>
-        <param name="multiplier">1</param>
-        <command_interface name="position">
-          <param name="min">0.0</param>
-          <param name="max">0.085</param>
-        </command_interface>
-        <command_interface name="velocity">
-          <param name="min">0.013</param>
-          <param name="max">0.1</param>
-        </command_interface>
-        <command_interface name="force">
-          <param name="min">5.0</param>
-          <param name="max">220.0</param>
-        </command_interface>
-        <state_interface name="position"/>
-        <state_interface name="velocity"/>
-        <state_interface name="force"/>
-      </joint>
-      <joint name="${prefix}robotiq_85_left_finger_tip_joint">
-        <param name="mimic">${prefix}robotiq_85_left_knuckle_joint</param>
-        <param name="multiplier">-1</param>
-        <command_interface name="position">
-          <param name="min">0.0</param>
-          <param name="max">0.085</param>
-        </command_interface>
-        <command_interface name="velocity">
-          <param name="min">0.013</param>
-          <param name="max">0.1</param>
-        </command_interface>
-        <command_interface name="force">
-          <param name="min">5.0</param>
-          <param name="max">220.0</param>
-        </command_interface>
-        <state_interface name="position"/>
-        <state_interface name="velocity"/>
-        <state_interface name="force"/>
-      </joint>
-      <joint name="${prefix}robotiq_85_right_finger_tip_joint">
-        <param name="mimic">${prefix}robotiq_85_left_knuckle_joint</param>
-        <param name="multiplier">-1</param>
-        <command_interface name="position">
-          <param name="min">0.0</param>
-          <param name="max">0.085</param>
-        </command_interface>
-        <command_interface name="velocity">
-          <param name="min">0.013</param>
-          <param name="max">0.1</param>
-        </command_interface>
-        <command_interface name="force">
-          <param name="min">5.0</param>
-          <param name="max">220.0</param>
-        </command_interface>
-        <state_interface name="position"/>
-        <state_interface name="velocity"/>
-        <state_interface name="force"/>
-      </joint>
-    </ros2_control>
   </xacro:macro>
 </robot>

Commit message: Update code to the newest nomenclature and state.

File: robotiq_85_description/urdf/robotiq_85_gripper.ros2_control.xacro (robot description, xacro)
@@ -4,23 +4,23 @@
     name
     prefix
-    use_fake_hardware:=false
-    fake_sensor_commands:=false
-    sim_gazebo:=false
-    sim_ignition:=false">
+    use_mock_hardware:=false
+    mock_sensor_commands:=false
+    sim_gazebo_classic:=false
+    sim_gazebo:=false">
 <!-- NOTE - currently using "system" because it is only supported hardware_interface-type by Gazebo and Ignition -->
     <ros2_control name="${name}" type="system">
       <hardware>
-        <xacro:if value="${sim_gazebo}">
+        <xacro:if value="${sim_gazebo_classic}">
           <plugin>gazebo_ros2_control/GazeboSystem</plugin>
         </xacro:if>
-        <xacro:if value="${sim_ignition}">
+        <xacro:if value="${sim_gazebo}">
           <plugin>ign_ros2_control/IgnitionSystem</plugin>
         </xacro:if>
-        <xacro:if value="${use_fake_hardware}">
+        <xacro:if value="${use_mock_hardware}">
           <plugin>fake_components/GenericSystem</plugin>
-          <param name="fake_sensor_commands">${fake_sensor_commands}</param>
+          <param name="mock_sensor_commands">${mock_sensor_commands}</param>
           <param name="state_following_offset">0.0</param>
         </xacro:if>
-        <xacro:unless value="${use_fake_hardware or sim_gazebo or sim_ignition}">
+        <xacro:unless value="${use_mock_hardware or sim_gazebo_classic or sim_gazebo}">
           <plugin>robotiq_hardware_interface/NOT_IMPLEMENTED_YET</plugin>
           <param name="ADD_GRIPPER_RELEVANT_PARAMETERS">654321</param>

File: robotiq_85_description/urdf/robotiq_85_gripper_macro.urdf.xacro (robot description, xacro)
@@ -8,21 +8,21 @@
     parent
     *origin
-    use_fake_hardware:=false
-    fake_sensor_commands:=false
-    sim_gazebo:=false
-    sim_ignition:=false">
+    use_mock_hardware:=false
+    mock_sensor_commands:=false
+    sim_gazebo_classic:=false
+    sim_gazebo:=false">
     <!-- The current hardware driver does not depend on ros2_control but we do utilize
     it for simulating the gripper with FakeSystem, Gazebo and  Igntion. Enabling this on
     hardware causes the JointStateBroadcaster to publish values for all joints including
     ones that are mimic'd which is causing issues on systems consuming the joint_state data. -->
-    <xacro:if value="${use_fake_hardware or sim_gazebo or sim_ignition}">
+    <xacro:if value="${use_mock_hardware or sim_gazebo_classic or sim_gazebo}">
       <!-- ros2 control instance -->
       <xacro:robotiq_85_gripper_ros2_control
         name="${name}"
         prefix="${prefix}"
-        use_fake_hardware="${use_fake_hardware}"
-        fake_sensor_commands="${fake_sensor_commands}"
+        use_mock_hardware="${use_mock_hardware}"
+        mock_sensor_commands="${mock_sensor_commands}"
+        sim_gazebo_classic="${sim_gazebo_classic}"
         sim_gazebo="${sim_gazebo}"
-        sim_ignition="${sim_ignition}"
         />
     </xacro:if>
@@ -33,5 +33,5 @@
     </joint>
     <link name="${prefix}robotiq_85_base_link">
-      <xacro:unless value="${sim_ignition}">
+      <xacro:unless value="${sim_gazebo}">
         <!-- Visual aid for grasping -->
         <visual>
@@ -113,7 +113,7 @@
         <mass value="0.018491" />
         <origin xyz="0.0 0.0 0.0" />
-        <inertia ixx = "0.000009" ixy = "-0.000001" ixz = "0.000000"
-          iyx = "-0.000001" iyy = "0.000001" iyz = "0.000000"
-          izx = "0.000000" izy = "0.000000" izz = "0.000010" />
+        <inertia ixx = "0.0009" ixy = "-0.0001" ixz = "0.000000"
+                 iyx = "-0.0001" iyy = "0.0001" iyz = "0.000000"
+                 izx = "0.000000" izy = "0.000000" izz = "0.0010" />
       </inertial>
     </link>
@@ -132,7 +132,7 @@
         <mass value="0.018491" />
         <origin xyz="0.0 0.0 0.0" />
-        <inertia ixx = "0.000009" ixy = "-0.000001" ixz = "0.000000"
-          iyx = "-0.000001" iyy = "0.000001" iyz = "0.000000"
-          izx = "0.000000" izy = "0.000000" izz = "0.000010" />
+        <inertia ixx = "0.0009" ixy = "-0.0001" ixz = "0.000000"
+                 iyx = "-0.0001" iyy = "0.0001" iyz = "0.000000"
+                 izx = "0.000000" izy = "0.000000" izz = "0.0010" />
       </inertial>
     </link>
